File: Nexus_links_pcb1.brd (EAGLE design)
At the start: 19 x 99.6 mm, 42 parts, among them IC1 TL074D, IC4 TL074D, J1 PJ301_THONKICONN6, J10 PJ301_THONKICONN6, J11 PJ301_THONKICONN6, J12 PJ301_THONKICONN6, J2 PJ301_THONKICONN6, J3 PJ301_THONKICONN6, J4 PJ301_THONKICONN6, J5 PJ301_THONKICONN6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

Commit message: updated in december
Parts:
- C1, C2: value 4.7u -> 10u
Changed lines of the file:
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@@
 <attribute name="VALUE" x="18.994475" y="73.739375" size="0.4064" layer="27" rot="R270"/>
 </element>
-<element name="C1" library="rcl" package="PANASONIC_A" value="4.7u" x="12.144375" y="87.78875" smashed="yes" rot="R270">
+<element name="C1" library="rcl" package="PANASONIC_A" value="10u" x="12.144375" y="87.78875" smashed="yes" rot="R270">
 <attribute name="NAME" x="11.509375" y="90.32875" size="0.6096" layer="25"/>
+<attribute name="RSPARTNUMBER" value="568-711" x="12.144375" y="87.78875" size="1.778" layer="27" rot="R270" display="off"/>
 <attribute name="VALUE" x="11.509375" y="90.96375" size="0.4064" layer="27"/>
 </element>
-<element name="C2" library="rcl" package="PANASONIC_A" value="4.7u" x="8.493125" y="87.78875" smashed="yes" rot="R270">
+<element name="C2" library="rcl" package="PANASONIC_A" value="10u" x="8.493125" y="87.78875" smashed="yes" rot="R270">
 <attribute name="NAME" x="7.858125" y="90.32875" size="0.6096" layer="25"/>
+<attribute name="RSPARTNUMBER" value="568-711" x="8.493125" y="87.78875" size="1.778" layer="27" rot="R270" display="off"/>
 <attribute name="VALUE" x="7.858125" y="90.96375" size="0.4064" layer="27"/>
 </element>
@@
 <element name="C3" library="rcl" package="C0603" value="100n" x="16.98625" y="56.35625" smashed="yes" rot="R180">
 <attribute name="NAME" x="17.30375" y="55.72135" size="0.6096" layer="25" rot="R180"/>
+<attribute name="RSPARTNUMBER" value="264-4416" x="16.98625" y="56.35625" size="1.778" layer="27" rot="R180" display="off"/>
 <attribute name="VALUE" x="17.30375" y="55.08635" size="0.4064" layer="27" rot="R180"/>
 </element>
 <element name="D2" library="diode" package="SOD123" value="1N5819HW" x="17.383125" y="86.99505" smashed="yes" rot="R270">
 <attribute name="NAME" x="16.383125" y="85.89525" size="0.6096" layer="25" rot="R90"/>
+<attribute name="RSPARTNUMBER" value="708-2197" x="17.383125" y="86.99505" size="1.778" layer="27" rot="R270" display="off"/>
 </element>
 <element name="D1" library="diode" package="SOD123" value="1N5819HW" x="2.143125" y="86.598175" smashed="yes" rot="R90">
 <attribute name="NAME" x="1.143225" y="85.498075" size="0.6096" layer="25" rot="R90"/>
+<attribute name="RSPARTNUMBER" value="708-2197" x="2.143125" y="86.598175" size="1.778" layer="27" rot="R90" display="off"/>
 <attribute name="VALUE" x="1.109325" y="86.609375" size="0.4064" layer="27" rot="R90"/>
 </element>
 <element name="LED1" library="led" package="LED3MM" value="L-937GYW" x="14.5" y="83.5" smashed="yes" rot="MR180">
 <attribute name="NAME" x="12.75375" y="81.1823" size="0.6096" layer="26" ratio="10" rot="MR0"/>
+<attribute name="RSPARTNUMBER" value="228-5663 " x="14.5" y="83.5" size="1.778" layer="28" rot="MR180" display="off"/>
 <attribute name="VALUE" x="8.4674" y="81.5315" size="0.4064" layer="28" ratio="10" rot="MR0"/>
 </element>
@@
 <element name="LED3" library="led" package="LED3MM" value="L-937GYW" x="4.5" y="32" smashed="yes" rot="MR180">
 <attribute name="NAME" x="1.245525" y="29.952125" size="0.6096" layer="26" ratio="10" rot="MR180"/>
+<attribute name="RSPARTNUMBER" value="228-5663 " x="4.5" y="32" size="1.778" layer="28" rot="MR180" display="off"/>
 <attribute name="VALUE" x="4.738125" y="29.285375" size="0.4064" layer="28" ratio="10" rot="MR180"/>
 </element>
@@
 <element name="C9" library="rcl" package="C0603" value="10p" x="10.080675" y="34.686925" smashed="yes" rot="R180">
 <attribute name="NAME" x="11.668175" y="35.163125" size="0.6096" layer="25" rot="R270"/>
+<attribute name="RSPARTNUMBER" value="601-0198 " x="10.080675" y="34.686925" size="1.778" layer="27" rot="R180" display="off"/>
 <attribute name="VALUE" x="12.303275" y="35.321825" size="0.4064" layer="27" rot="R90"/>
 </element>

Commit message: updated values to precission adder
Parts:
- R15: value 33k -> 100k
Changed lines of the file:
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@@
 <?xml version="1.0" encoding="utf-8"?>
 <!DOCTYPE eagle SYSTEM "eagle.dtd">
-<eagle version="8.7.0">
+<eagle version="9.2.2">
 <drawing>
 <settings>
@@
 <param name="checkStop" value="0"/>
 <param name="checkValues" value="0"/>
+<param name="checkNames" value="1"/>
+<param name="checkWireStubs" value="1"/>
+<param name="checkPolygonWidth" value="0"/>
 <param name="useDiameter" value="13"/>
 <param name="maxErrors" value="50"/>
@@
 <attribute name="VALUE" x="12.303275" y="35.321825" size="0.4064" layer="27" rot="R90"/>
 </element>
-<element name="R15" library="rcl" package="R0603" value="33k" x="6.145" y="35.361825" smashed="yes">
+<element name="R15" library="rcl" package="R0603" value="100k" x="6.145" y="35.361825" smashed="yes">
 <attribute name="NAME" x="7.4151" y="34.568025" size="0.6096" layer="25" rot="R180"/>
 <attribute name="VALUE" x="7.415" y="33.933025" size="0.4064" layer="27" rot="R180"/>
@@
 <attribute name="VALUE" x="2.143125" y="48.656925" size="0.4064" layer="27"/>
 </element>
-<element name="U$2" library="og-pcb-art" package="ROHS" value="" x="4.089325" y="73.068175"/>
+<element name="U$2" library="og-pcb-art" package="ROHS" value="" x="4.089325" y="73.068175" smashed="yes"/>
 <element name="J1" library="og-pj301" package="WQP_PJ_301M6" value="PJ301_THONKICONN6" x="4.5" y="83.5" smashed="yes" rot="MR180">
 <attribute name="NAME" x="2.1737" y="88.3414" size="1.27" layer="26" rot="MR0"/>
@@
 <attribute name="NAME" x="9" y="10.8412" size="1.27" layer="26" rot="MR0"/>
 </element>
-<element name="R6" library="rcl" package="R0603" value="51" x="2.04" y="59.928125"/>
-<element name="J5" library="og-pj301" package="WQP_PJ_301M6" value="PJ301_THONKICONN6" x="4.5" y="58" rot="MR0"/>
-<element name="R7" library="rcl" package="R0603" value="100k" x="16.748125" y="4.28625"/>
-<element name="J6" library="og-pj301" package="WQP_PJ_301M6" value="PJ301_THONKICONN6" x="14.5" y="6" rot="MR180"/>
+<element name="R6" library="rcl" package="R0603" value="51" x="2.04" y="59.928125" smashed="yes">
+<attribute name="NAME" x="1.405" y="60.563125" size="1.27" layer="25"/>
+<attribute name="VALUE" x="1.405" y="58.023125" size="1.27" layer="27"/>
+</element>
+<element name="J5" library="og-pj301" package="WQP_PJ_301M6" value="PJ301_THONKICONN6" x="4.5" y="58" smashed="yes" rot="MR0">
+<attribute name="NAME" x="0" y="53" size="1.27" layer="26" rot="MR180"/>
+</element>
+<element name="R7" library="rcl" package="R0603" value="100k" x="16.748125" y="4.28625" smashed="yes">
+<attribute name="NAME" x="16.113125" y="4.92125" size="1.27" layer="25"/>
+<attribute name="VALUE" x="16.113125" y="2.38125" size="1.27" layer="27"/>
+</element>
+<element name="J6" library="og-pj301" package="WQP_PJ_301M6" value="PJ301_THONKICONN6" x="14.5" y="6" smashed="yes" rot="MR180">
+<attribute name="NAME" x="19" y="11" size="1.27" layer="26" rot="MR0"/>
+</element>
 </elements>
 <signals>
@@
 </signal>
 </signals>
+<mfgpreviewcolors>
+<mfgpreviewcolor name="soldermaskcolor" color="0xC8008000"/>
+<mfgpreviewcolor name="silkscreencolor" color="0xFFFEFEFE"/>
+<mfgpreviewcolor name="backgroundcolor" color="0xFF282828"/>
+<mfgpreviewcolor name="coppercolor" color="0xFFFFBF00"/>
+<mfgpreviewcolor name="substratecolor" color="0xFF786E46"/>
+</mfgpreviewcolors>
 </board>
 </drawing>
